File: texas-blinky.kicad_pcb (KiCad board)
At the start: 2 copper layers, 62 x 60.3 mm, 6 parts, among them Q1 MMBT3904

Commit message: Update R1 value to 100k in PCB, rotate for battery clearance
Co-Authored-By: Claude Sonnet 4.6 <noreply@anthropic.com>
Parts:
- R1: value 1M -> 100k
- moved R2 6.84 mm to (114.3, 62.2), turned to 90 degrees
Routing:
- net Net-(D1-A): track 25.6 -> 34.8 mm
- net Net-(BT1-+): track 56.3 -> 50.3 mm
Changed lines of the file:
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@@
 	(footprint "Resistor_THT:R_Axial_DIN0207_L6.3mm_D2.5mm_P7.62mm_Horizontal"
 		(layer "F.Cu")
-		(at 116.84 55.88)
+		(at 114.3 62.23 90)
 		(descr "Resistor, Axial_DIN0207 series, Axial, Horizontal, pin pitch=7.62mm, 0.25W = 1/4W, length*diameter=6.3*2.5mm^2, http://cdn-reichelt.de/documents/datenblatt/B400/1_4W%23YAG.pdf")
 		(tags "Resistor Axial_DIN0207 series Axial Horizontal pin pitch 7.62mm 0.25W = 1/4W length 6.3mm diameter 2.5mm")
 		(property "Reference" "R2"
-			(at 3.81 -2.37 0)
+			(at 3.81 -2.37 90)
 			(layer "F.SilkS")
 			(effects
@@
 		)
 		(property "Value" "100R"
-			(at 3.81 2.37 0)
+			(at 3.81 2.37 90)
 			(layer "F.Fab")
 			(effects
@@
 		)
 		(property "Datasheet" "~"
-			(at 0 0 0)
+			(at 0 0 90)
 			(layer "F.Fab")
 			(hide yes)
@@
 		)
 		(property "Description" "Resistor"
-			(at 0 0 0)
+			(at 0 0 90)
 			(layer "F.Fab")
 			(hide yes)
@@
 		(attr through_hole)
 		(fp_line
+			(start 7.08 -1.37)
+			(end 7.08 -1.04)
+			(stroke
+				(width 0.12)
+				(type solid)
+			)
+			(layer "F.SilkS")
+		)
+		(fp_line
 			(start 0.54 -1.37)
 			(end 7.08 -1.37)
@@
 		)
 		(fp_line
+			(start 7.08 1.37)
+			(end 7.08 1.04)
+			(stroke
+				(width 0.12)
+				(type solid)
+			)
+			(layer "F.SilkS")
+		)
+		(fp_line
 			(start 0.54 1.37)
 			(end 7.08 1.37)
-			(stroke
-				(width 0.12)
-				(type solid)
-			)
-			(layer "F.SilkS")
-		)
-		(fp_line
-			(start 7.08 -1.37)
-			(end 7.08 -1.04)
-			(stroke
-				(width 0.12)
-				(type solid)
-			)
-			(layer "F.SilkS")
-		)
-		(fp_line
-			(start 7.08 1.37)
-			(end 7.08 1.04)
 			(stroke
 				(width 0.12)
@@
 		)
 		(fp_line
+			(start 7.62 0)
+			(end 6.96 0)
+			(stroke
+				(width 0.1)
+				(type solid)
+			)
+			(layer "F.Fab")
+		)
+		(fp_line
 			(start 0 0)
 			(end 0.66 0)
-			(stroke
-				(width 0.1)
-				(type solid)
-			)
-			(layer "F.Fab")
-		)
-		(fp_line
-			(start 7.62 0)
-			(end 6.96 0)
 			(stroke
 				(width 0.1)
@@
 		)
 		(fp_text user "${REFERENCE}"
-			(at 3.81 0 0)
+			(at 3.81 0 90)
 			(layer "F.Fab")
 			(effects
@@
 		)
 		(pad "1" thru_hole circle
-			(at 0 0)
+			(at 0 0 90)
 			(size 1.6 1.6)
 			(drill 0.8)
@@
 		)
 		(pad "2" thru_hole circle
-			(at 7.62 0)
+			(at 7.62 0 90)
 			(size 1.6 1.6)
 			(drill 0.8)
@@
 			)
 		)
-		(property "Value" "1M"
+		(property "Value" "100k"
 			(at 3.81 2.37 90)
 			(layer "F.Fab")
@@
 	)
 	(segment
-		(start 116.015 66.04)
-		(end 116.015 56.705)
+		(start 111.76 78.74)
+		(end 114.3 76.2)
 		(width 0.2)
 		(layer "B.Cu")
@@
 	)
 	(segment
-		(start 111.76 78.74)
-		(end 114.3 76.2)
+		(start 114.3 64.325)
+		(end 116.015 66.04)
 		(width 0.2)
 		(layer "B.Cu")
@@
 	)
 	(segment
-		(start 116.015 56.705)
-		(end 116.84 55.88)
+		(start 114.3 76.2)
+		(end 116.015 76.2)
 		(width 0.2)
 		(layer "B.Cu")
@@
 	)
 	(segment
-		(start 114.3 76.2)
-		(end 116.015 76.2)
+		(start 114.3 62.23)
+		(end 114.3 64.325)
 		(width 0.2)
 		(layer "B.Cu")
@@
 	)
 	(segment
-		(start 124.46 58.42)
-		(end 137.16 71.12)
+		(start 114.3 54.61)
+		(end 130.81 71.12)
 		(width 0.2)
 		(layer "F.Cu")
@@
 	)
 	(segment
-		(start 124.46 55.88)
-		(end 124.46 58.42)
-		(width 0.2)
-		(layer "F.Cu")
-		(net 5)
-	)
-	(segment
-		(start 137.16 71.12)
+		(start 130.81 71.12)
 		(end 142.24 71.12)
 		(width 0.2)
